Commit message: Fix relative mesh paths

File: arm/vx300s.urdf (robot description, URDF)
Before this commit: robot vx300s, 14 links, 13 joints
Links:
- removed link vx300s/base_link
- removed link vx300s/ee_arm_link
- removed link vx300s/ee_gripper_link
- removed link vx300s/fingers_link
- removed link vx300s/gripper_bar_link
- removed link vx300s/gripper_link
- removed link vx300s/gripper_prop_link
- removed link vx300s/left_finger_link
- removed link vx300s/lower_forearm_link
- removed link vx300s/right_finger_link
- removed link vx300s/shoulder_link
- removed link vx300s/upper_arm_link
- removed link vx300s/upper_forearm_link
- removed link vx300s/wrist_link
- added link vx300s_base_link, mass 0.969034; collision mesh filename=./meshes/vx300s_meshes/vx300s_1_base.stl scale=0.001 0.001 0.001; visual mesh filename=./meshes/vx300s_meshes/vx300s_1_base.stl scale=0.001 0.001 0.001
- added link vx300s_ee_arm_link, mass 0.001
- added link vx300s_ee_gripper_link, mass 0.001
- added link vx300s_fingers_link, mass 0.001
- added link vx300s_gripper_bar_link, mass 0.150986; collision mesh filename=./meshes/vx300s_meshes/vx300s_9_gripper_bar.stl scale=0.001 0.001 0.001; visual mesh filename=./meshes/vx300s_meshes/vx300s_9_gripper_bar.stl scale=0.001 0.001 0.001
- added link vx300s_gripper_link, mass 0.097666; collision mesh filename=./meshes/vx300s_meshes/vx300s_7_gripper.stl scale=0.001 0.001 0.001; visual mesh filename=./meshes/vx300s_meshes/vx300s_7_gripper.stl scale=0.001 0.001 0.001
- added link vx300s_gripper_prop_link, mass 0.008009; collision mesh filename=./meshes/vx300s_meshes/vx300s_8_gripper_prop.stl scale=0.001 0.001 0.001; visual mesh filename=./meshes/vx300s_meshes/vx300s_8_gripper_prop.stl scale=0.001 0.001 0.001
- added link vx300s_left_finger_link, mass 0.034796; collision mesh filename=./meshes/vx300s_meshes/vx300s_10_gripper_finger.stl scale=0.001 0.001 0.001; visual mesh filename=./meshes/vx300s_meshes/vx300s_10_gripper_finger.stl scale=0.001 0.001 0.001
- added link vx300s_lower_forearm_link, mass 0.414823; collision mesh filename=./meshes/vx300s_meshes/vx300s_5_lower_forearm.stl scale=0.001 0.001 0.001; visual mesh filename=./meshes/vx300s_meshes/vx300s_5_lower_forearm.stl scale=0.001 0.001 0.001
- added link vx300s_right_finger_link, mass 0.034796; collision mesh filename=./meshes/vx300s_meshes/vx300s_10_gripper_finger.stl scale=0.001 0.001 0.001; visual mesh filename=./meshes/vx300s_meshes/vx300s_10_gripper_finger.stl scale=0.001 0.001 0.001
- added link vx300s_shoulder_link, mass 0.798614; collision mesh filename=./meshes/vx300s_meshes/vx300s_2_shoulder.stl scale=0.001 0.001 0.001; visual mesh filename=./meshes/vx300s_meshes/vx300s_2_shoulder.stl scale=0.001 0.001 0.001
- added link vx300s_upper_arm_link, mass 0.792592; collision mesh filename=./meshes/vx300s_meshes/vx300s_3_upper_arm.stl scale=0.001 0.001 0.001; visual mesh filename=./meshes/vx300s_meshes/vx300s_3_upper_arm.stl scale=0.001 0.001 0.001
- added link vx300s_upper_forearm_link, mass 0.322228; collision mesh filename=./meshes/vx300s_meshes/vx300s_4_upper_forearm.stl scale=0.001 0.001 0.001; visual mesh filename=./meshes/vx300s_meshes/vx300s_4_upper_forearm.stl scale=0.001 0.001 0.001
- added link vx300s_wrist_link, mass 0.115395; collision mesh filename=./meshes/vx300s_meshes/vx300s_6_wrist.stl scale=0.001 0.001 0.001; visual mesh filename=./meshes/vx300s_meshes/vx300s_6_wrist.stl scale=0.001 0.001 0.001
Joints:
- joint ee_arm: child vx300s/ee_arm_link -> vx300s_ee_arm_link; parent vx300s/gripper_link -> vx300s_gripper_link
- joint ee_bar: child vx300s/fingers_link -> vx300s_fingers_link; parent vx300s/gripper_bar_link -> vx300s_gripper_bar_link
- joint ee_gripper: child vx300s/ee_gripper_link -> vx300s_ee_gripper_link; parent vx300s/fingers_link -> vx300s_fingers_link
- joint elbow: child vx300s/upper_forearm_link -> vx300s_upper_forearm_link; parent vx300s/upper_arm_link -> vx300s_upper_arm_link
- joint forearm_roll: child vx300s/lower_forearm_link -> vx300s_lower_forearm_link; parent vx300s/upper_forearm_link -> vx300s_upper_forearm_link
- joint gripper: child vx300s/gripper_prop_link -> vx300s_gripper_prop_link; parent vx300s/ee_arm_link -> vx300s_ee_arm_link
- joint gripper_bar: child vx300s/gripper_bar_link -> vx300s_gripper_bar_link; parent vx300s/ee_arm_link -> vx300s_ee_arm_link
- joint left_finger: child vx300s/left_finger_link -> vx300s_left_finger_link; parent vx300s/fingers_link -> vx300s_fingers_link
- joint right_finger: child vx300s/right_finger_link -> vx300s_right_finger_link; parent vx300s/fingers_link -> vx300s_fingers_link
- joint shoulder: child vx300s/upper_arm_link -> vx300s_upper_arm_link; parent vx300s/shoulder_link -> vx300s_shoulder_link
- joint waist: child vx300s/shoulder_link -> vx300s_shoulder_link; parent vx300s/base_link -> vx300s_base_link
- joint wrist_angle: child vx300s/wrist_link -> vx300s_wrist_link; parent vx300s/lower_forearm_link -> vx300s_lower_forearm_link
- joint wrist_rotate: child vx300s/gripper_link -> vx300s_gripper_link; parent vx300s/wrist_link -> vx300s_wrist_link

Commit message: Trim the base

File: arm/vx300s.urdf (robot description, URDF)
Before this commit: robot vx300s, 14 links, 13 joints
Links:
- link vx300s_base_link: geometry collision mesh filename=./meshes/vx300s_meshes/vx300s_1_base_trimmed.stl scale=0.001 0.001 0.001; visual mesh filename=./meshes/vx300s_meshes/vx300s_1_base_trimmed.stl scale=0.001 0.001 0.001
