Commit message: Rename arm joints

File: go2_arm.urdf (robot description, URDF)
Before this commit: robot go2_with_arm, 52 links, 51 joints
Joints:
- removed joint arm_ee_bar
- removed joint arm_elbow
- removed joint arm_forearm_roll
- removed joint arm_gripper_bar
- removed joint arm_mount
- removed joint arm_shoulder
- removed joint arm_waist
- removed joint arm_wrist_angle
- removed joint arm_wrist_rotate
- added joint ee_bar_arm_joint: type fixed, parent vx300s_gripper_bar_link, child vx300s_fingers_link, origin xyz=0.025875 0 0 rpy=0 0 0, axis 1 0 0
- added joint elbow_arm_joint: type revolute, parent vx300s_upper_arm_link, child vx300s_upper_forearm_link, origin xyz=0.05955 0 0.3 rpy=0 0 0, axis 0 1 0, limit lower=-1.7627825445142729 upper=1.6057029118347832 effort=15 velocity=3.141592653589793
- added joint forearm_roll_arm_joint: type revolute, parent vx300s_upper_forearm_link, child vx300s_lower_forearm_link, origin xyz=0.2 0 0 rpy=0 0 0, axis 1 0 0, limit lower=-3.141582653589793 upper=3.141582653589793 effort=2 velocity=3.141592653589793
- added joint gripper_bar_arm_joint: type fixed, parent vx300s_ee_arm_link, child vx300s_gripper_bar_link, origin xyz=0 0 0 rpy=0 0 0, axis 1 0 0
- added joint mount_arm_joint: type fixed, parent base, child vx300s_base_link, origin xyz=0.0 0.0 0.05 rpy=0 0 0
- added joint shoulder_arm_joint: type revolute, parent vx300s_shoulder_link, child vx300s_upper_arm_link, origin xyz=0 0 0.04805 rpy=0 0 0, axis 0 1 0, limit lower=-1.8500490071139892 upper=1.2566370614359172 effort=20 velocity=3.141592653589793
- added joint waist_arm_joint: type revolute, parent vx300s_base_link, child vx300s_shoulder_link, origin xyz=0 0 0.079 rpy=0 0 0, axis 0 0 1, limit lower=-3.141582653589793 upper=3.141582653589793 effort=10 velocity=3.141592653589793
- added joint wrist_angle_arm_joint: type revolute, parent vx300s_lower_forearm_link, child vx300s_wrist_link, origin xyz=0.1 0 0 rpy=0 0 0, axis 0 1 0, limit lower=-1.8675022996339325 upper=2.234021442552742 effort=5 velocity=3.141592653589793
- added joint wrist_rotate_arm_joint: type revolute, parent vx300s_wrist_link, child vx300s_gripper_link, origin xyz=0.069744 0 0 rpy=0 0 0, axis 1 0 0, limit lower=-3.141582653589793 upper=3.141582653589793 effort=1 velocity=3.141592653589793

Commit message: Remove fingers link

File: go2_arm.urdf (robot description, URDF)
Before this commit: robot go2_with_arm, 52 links, 51 joints
Links:
- removed link vx300s_fingers_link
Joints:
- joint ee_bar_arm_joint: child vx300s_fingers_link -> (none)

Commit message: Remove the redundant ee_bar_arm_joint

File: go2_arm.urdf (robot description, URDF)
Before this commit: robot go2_with_arm, 51 links, 51 joints
Joints:
- removed joint ee_bar_arm_joint

Commit message: Disable collisions for the arm

File: go2_arm.urdf (robot description, URDF)
Before this commit: robot go2_with_arm, 51 links, 50 joints
Links:
- link vx300s_base_link: geometry visual mesh filename=./meshes/vx300s_meshes/vx300s_1_base_trimmed.stl scale=0.001 0.001 0.001
- link vx300s_gripper_bar_link: geometry visual mesh filename=./meshes/vx300s_meshes/vx300s_9_gripper_bar.stl scale=0.001 0.001 0.001
- link vx300s_gripper_link: geometry visual mesh filename=./meshes/vx300s_meshes/vx300s_7_gripper.stl scale=0.001 0.001 0.001
- link vx300s_lower_forearm_link: geometry visual mesh filename=./meshes/vx300s_meshes/vx300s_5_lower_forearm.stl scale=0.001 0.001 0.001
- link vx300s_shoulder_link: geometry visual mesh filename=./meshes/vx300s_meshes/vx300s_2_shoulder.stl scale=0.001 0.001 0.001
- link vx300s_upper_arm_link: geometry visual mesh filename=./meshes/vx300s_meshes/vx300s_3_upper_arm.stl scale=0.001 0.001 0.001
- link vx300s_upper_forearm_link: geometry visual mesh filename=./meshes/vx300s_meshes/vx300s_4_upper_forearm.stl scale=0.001 0.001 0.001
- link vx300s_wrist_link: geometry visual mesh filename=./meshes/vx300s_meshes/vx300s_6_wrist.stl scale=0.001 0.001 0.001

Commit message: More rotation to the wrist

File: go2_arm.urdf (robot description, URDF)
Before this commit: robot go2_with_arm, 51 links, 50 joints
Joints:
- joint wrist_rotate_arm_joint: limit lower=-3.141582653589793 upper=3.141582653589793 effort=1 velocity=3.141592653589793 -> lower=-6.28318530718 upper=6.28318530718 effort=1 velocity=3.141592653589793
