Commit message: Resize thigh boxes

File: go2_arm_dummy.urdf (robot description, URDF)
Before this commit: robot go2_with_arm, 39 links, 38 joints
Links:
- link FL_thigh: geometry collision box size=0.213 0.0245 0.034; visual mesh filename=./dae/thigh.dae
- link FR_thigh: geometry collision box size=0.213 0.0245 0.034; visual mesh filename=./dae/thigh_mirror.dae
- link RL_thigh: geometry collision box size=0.213 0.0245 0.034; visual mesh filename=./dae/thigh.dae
- link RR_thigh: geometry collision box size=0.213 0.0245 0.034; visual mesh filename=./dae/thigh_mirror.dae
