Commit message: Massless arm with fixed joints except for the revolute wrist

File: go2_arm_fixed.urdf (robot description, URDF)
Before this commit: robot go2_with_arm, 51 links, 50 joints
Links:
- link vx300s_base_link: mass 0.969034 -> 0
- link vx300s_ee_arm_link: mass 0.001 -> 0
- link vx300s_gripper_bar_link: mass 0.150986 -> 0
- link vx300s_gripper_link: mass 0.097666 -> 0
- link vx300s_lower_forearm_link: mass 0.414823 -> 0
- link vx300s_shoulder_link: mass 0.798614 -> 0
- link vx300s_upper_arm_link: mass 0.792592 -> 0
- link vx300s_upper_forearm_link: mass 0.322228 -> 0
- link vx300s_wrist_link: mass 0.115395 -> 0
Joints:
- joint wrist_angle_arm_joint: type fixed -> revolute

Commit message: Remove rotors

File: go2_arm_fixed.urdf (robot description, URDF)
Before this commit: robot go2_with_arm, 51 links, 50 joints
Links:
- removed link FL_calf_rotor
- removed link FL_hip_rotor
- removed link FL_thigh_rotor
- removed link FR_calf_rotor
- removed link FR_hip_rotor
- removed link FR_thigh_rotor
- removed link RL_calf_rotor
- removed link RL_hip_rotor
- removed link RL_thigh_rotor
- removed link RR_calf_rotor
- removed link RR_hip_rotor
- removed link RR_thigh_rotor
Joints:
- removed joint FL_calf_rotor_joint
- removed joint FL_hip_rotor_joint
- removed joint FL_thigh_rotor_joint
- removed joint FR_calf_rotor_joint
- removed joint FR_hip_rotor_joint
- removed joint FR_thigh_rotor_joint
- removed joint RL_calf_rotor_joint
- removed joint RL_hip_rotor_joint
- removed joint RL_thigh_rotor_joint
- removed joint RR_calf_rotor_joint
- removed joint RR_hip_rotor_joint
- removed joint RR_thigh_rotor_joint

Commit message: Replace vx300s arm with the low cost arm, which is much smaller

File: go2_arm_fixed.urdf (robot description, URDF)
Before this commit: robot go2_with_arm, 39 links, 38 joints
Links:
- removed link vx300s_base_link
- removed link vx300s_ee_arm_link
- removed link vx300s_gripper_bar_link
- removed link vx300s_gripper_link
- removed link vx300s_lower_forearm_link
- removed link vx300s_shoulder_link
- removed link vx300s_upper_arm_link
- removed link vx300s_upper_forearm_link
- removed link vx300s_wrist_link
- added link base_link, mass 0.06752363433035656; collision mesh filename=./meshes/base_link.stl scale=0.001 0.001 0.001; visual mesh filename=./meshes/base_link.stl scale=0.001 0.001 0.001
- added link elbow-to-wrist-motor-reference_v1_1, mass 0.02059907441055582; collision mesh filename=./meshes/elbow-to-wrist-motor-reference_v1_1.stl scale=0.001 0.001 0.001; visual mesh filename=./meshes/elbow-to-wrist-motor-reference_v1_1.stl scale=0.001 0.001 0.001
- added link first-bracket-motor_1, mass 0.050669759178187244; collision mesh filename=./meshes/first-bracket-motor_1.stl scale=0.001 0.001 0.001; visual mesh filename=./meshes/first-bracket-motor_1.stl scale=0.001 0.001 0.001
- added link gripper-moving-part-dumb_v2_1, mass 0.013583445641331692; collision mesh filename=./meshes/gripper-moving-part-dumb_v2_1.stl scale=0.001 0.001 0.001; visual mesh filename=./meshes/gripper-moving-part-dumb_v2_1.stl scale=0.001 0.001 0.001
- added link gripper-static-motor_v2_1, mass 0.030801959916802346; collision mesh filename=./meshes/gripper-static-motor_v2_1.stl scale=0.001 0.001 0.001; visual mesh filename=./meshes/gripper-static-motor_v2_1.stl scale=0.001 0.001 0.001
- added link shoulder-to-elbow-motor_v1_1, mass 0.05261369068977079; collision mesh filename=./meshes/shoulder-to-elbow-motor_v1_1.stl scale=0.001 0.001 0.001; visual mesh filename=./meshes/shoulder-to-elbow-motor_v1_1.stl scale=0.001 0.001 0.001
Joints:
- removed joint arm_ee_arm
- removed joint elbow_arm_joint
- removed joint forearm_roll_arm_joint
- removed joint gripper_bar_arm_joint
- added joint gripper_arm_joint: type fixed, parent gripper-static-motor_v2_1, child gripper-moving-part-dumb_v2_1, origin xyz=-0.00755 0.01299 0.01425 rpy=0 0 0, axis -0.0 -0.0 -1.0
- joint mount_arm_joint: child vx300s_base_link -> base_link; origin xyz=0.0 0.0 0.05 rpy=0 0 0 -> xyz=0.0 0.0 0.05 rpy=0 0 -1.57079
- joint shoulder_arm_joint: axis 0 1 0 -> 1.0 0.0 0.0; child vx300s_upper_arm_link -> shoulder-to-elbow-motor_v1_1; limit lower=-1.8500490071139892 upper=1.2566370614359172 effort=20 velocity=3.141592653589793 -> (none); origin xyz=0 0 0.04805 rpy=0 0 0 -> xyz=0.0192 0.0002 0.01425 rpy=0 0 0; parent vx300s_shoulder_link -> first-bracket-motor_1
- joint waist_arm_joint: axis 0 0 1 -> 0.0 0.0 1.0; child vx300s_shoulder_link -> first-bracket-motor_1; limit lower=-3.141582653589793 upper=3.141582653589793 effort=10 velocity=3.141592653589793 -> (none); origin xyz=0 0 0.079 rpy=0 0 0 -> xyz=0.00025 0.06875 0.0409 rpy=0 0 0; parent vx300s_base_link -> base_link
- joint wrist_angle_arm_joint: axis 0 1 0 -> 1.0 -0.0 0.0; child vx300s_wrist_link -> elbow-to-wrist-motor-reference_v1_1; limit lower=-1.8675022996339325 upper=2.234021442552742 effort=5 velocity=3.141592653589793 -> (none); origin xyz=0.1 0 0 rpy=0 0 0 -> xyz=-0.03375 0.0148 0.1083 rpy=0 0 0; parent vx300s_lower_forearm_link -> shoulder-to-elbow-motor_v1_1; type revolute -> fixed
- joint wrist_rotate_arm_joint: axis 1 0 0 -> -0.0 -1.0 0.0; child vx300s_gripper_link -> gripper-static-motor_v2_1; limit lower=-3.141582653589793 upper=3.141582653589793 effort=1 velocity=3.141592653589793 -> (none); origin xyz=0.069744 0 0 rpy=0 0 0 -> xyz=0.013407 0.044938 -1.3e-05 rpy=0 0 0; parent vx300s_wrist_link -> elbow-to-wrist-motor-reference_v1_1

Commit message: Refactor

File: go2_arm_fixed.urdf (robot description, URDF)
Before this commit: robot go2_with_arm, 36 links, 35 joints
Links:
- removed link elbow-to-wrist-motor-reference_v1_1
- removed link first-bracket-motor_1
- removed link gripper-moving-part-dumb_v2_1
- removed link gripper-static-motor_v2_1
- removed link shoulder-to-elbow-motor_v1_1
- added link elbow_to_wrist_motor_reference_v1_1, mass 0.02059907441055582; collision mesh filename=./meshes/elbow-to-wrist-motor-reference_v1_1.stl scale=0.001 0.001 0.001; visual mesh filename=./meshes/elbow-to-wrist-motor-reference_v1_1.stl scale=0.001 0.001 0.001
- added link first_bracket_motor_1, mass 0.050669759178187244; collision mesh filename=./meshes/first-bracket-motor_1.stl scale=0.001 0.001 0.001; visual mesh filename=./meshes/first-bracket-motor_1.stl scale=0.001 0.001 0.001
- added link gripper_moving_part_dumb_v2_1, mass 0.013583445641331692; collision mesh filename=./meshes/gripper-moving-part-dumb_v2_1.stl scale=0.001 0.001 0.001; visual mesh filename=./meshes/gripper-moving-part-dumb_v2_1.stl scale=0.001 0.001 0.001
- added link gripper_static_motor_v2_1, mass 0.030801959916802346; collision mesh filename=./meshes/gripper-static-motor_v2_1.stl scale=0.001 0.001 0.001; visual mesh filename=./meshes/gripper-static-motor_v2_1.stl scale=0.001 0.001 0.001
- added link shoulder_to_elbow_motor_v1_1, mass 0.05261369068977079; collision mesh filename=./meshes/shoulder-to-elbow-motor_v1_1.stl scale=0.001 0.001 0.001; visual mesh filename=./meshes/shoulder-to-elbow-motor_v1_1.stl scale=0.001 0.001 0.001
Joints:
- joint gripper_arm_joint: child gripper-moving-part-dumb_v2_1 -> gripper_moving_part_dumb_v2_1; parent gripper-static-motor_v2_1 -> gripper_static_motor_v2_1
- joint shoulder_arm_joint: child shoulder-to-elbow-motor_v1_1 -> shoulder_to_elbow_motor_v1_1; parent first-bracket-motor_1 -> first_bracket_motor_1
- joint waist_arm_joint: child first-bracket-motor_1 -> first_bracket_motor_1
- joint wrist_angle_arm_joint: child elbow-to-wrist-motor-reference_v1_1 -> elbow_to_wrist_motor_reference_v1_1; parent shoulder-to-elbow-motor_v1_1 -> shoulder_to_elbow_motor_v1_1
- joint wrist_rotate_arm_joint: child gripper-static-motor_v2_1 -> gripper_static_motor_v2_1; parent elbow-to-wrist-motor-reference_v1_1 -> elbow_to_wrist_motor_reference_v1_1

Commit message: Refactor encore

File: go2_arm_fixed.urdf (robot description, URDF)
Before this commit: robot go2_with_arm, 36 links, 35 joints
Links:
- link elbow_to_wrist_motor_reference_v1_1: geometry collision mesh filename=./meshes/elbow_to_wrist_motor_reference_v1_1.stl scale=0.001 0.001 0.001; visual mesh filename=./meshes/elbow_to_wrist_motor_reference_v1_1.stl scale=0.001 0.001 0.001
- link first_bracket_motor_1: geometry collision mesh filename=./meshes/first_bracket_motor_1.stl scale=0.001 0.001 0.001; visual mesh filename=./meshes/first_bracket_motor_1.stl scale=0.001 0.001 0.001
- link gripper_moving_part_dumb_v2_1: geometry collision mesh filename=./meshes/gripper_moving_part_dumb_v2_1.stl scale=0.001 0.001 0.001; visual mesh filename=./meshes/gripper_moving_part_dumb_v2_1.stl scale=0.001 0.001 0.001
- link gripper_static_motor_v2_1: geometry collision mesh filename=./meshes/gripper_static_motor_v2_1.stl scale=0.001 0.001 0.001; visual mesh filename=./meshes/gripper_static_motor_v2_1.stl scale=0.001 0.001 0.001
- link shoulder_to_elbow_motor_v1_1: geometry collision mesh filename=./meshes/shoulder_to_elbow_motor_v1_1.stl scale=0.001 0.001 0.001; visual mesh filename=./meshes/shoulder_to_elbow_motor_v1_1.stl scale=0.001 0.001 0.001

Commit message: Revolute joint for the wrist

File: go2_arm_fixed.urdf (robot description, URDF)
Before this commit: robot go2_with_arm, 36 links, 35 joints
Joints:
- joint wrist_angle_arm_joint: limit (none) -> lower=-1.0472 upper=1.0472 effort=23.7 velocity=30.1; type fixed -> revolute
