Commit message: The length of the thigh collision shape is shortened from 0.213 to 0.11

File: go2.urdf (robot description, URDF)
Before this commit: robot go2, 42 links, 41 joints
Links:
- link FL_thigh: geometry collision box size=0.11 0.0245 0.034; visual mesh filename=./dae/thigh.dae
- link FR_thigh: geometry collision box size=0.11 0.0245 0.034; visual mesh filename=./dae/thigh_mirror.dae
- link RL_thigh: geometry collision box size=0.11 0.0245 0.034; visual mesh filename=./dae/thigh.dae
- link RR_thigh: geometry collision box size=0.11 0.0245 0.034; visual mesh filename=./dae/thigh_mirror.dae

File: go2_arm.urdf (robot description, URDF)
Before this commit: robot go2_with_arm, 51 links, 50 joints
Links:
- link FL_thigh: geometry collision box size=0.11 0.0245 0.034; visual mesh filename=./dae/thigh.dae
- link FR_thigh: geometry collision box size=0.11 0.0245 0.034; visual mesh filename=./dae/thigh_mirror.dae
- link RL_thigh: geometry collision box size=0.11 0.0245 0.034; visual mesh filename=./dae/thigh.dae
- link RR_thigh: geometry collision box size=0.11 0.0245 0.034; visual mesh filename=./dae/thigh_mirror.dae

Commit message: drop-in replacement for solo12 urdf

File: go2.urdf (robot description, URDF)
Before this commit: robot go2, 42 links, 41 joints
Links:
- removed link FL_calf
- removed link FL_calf_rotor
- removed link FL_calflower
- removed link FL_calflower1
- removed link FL_hip
- removed link FL_hip_rotor
- removed link FL_thigh
- removed link FL_thigh_rotor
- removed link FR_calf
- removed link FR_calf_rotor
- removed link FR_calflower
- removed link FR_calflower1
- removed link FR_hip
- removed link FR_hip_rotor
- removed link FR_thigh
- removed link FR_thigh_rotor
- removed link RL_calf
- removed link RL_calf_rotor
- removed link RL_calflower
- removed link RL_calflower1
- removed link RL_foot
- removed link RL_hip
- removed link RL_hip_rotor
- removed link RL_thigh
- removed link RL_thigh_rotor
- removed link RR_calf
- removed link RR_calf_rotor
- removed link RR_calflower
- removed link RR_calflower1
- removed link RR_foot
- removed link RR_hip
- removed link RR_hip_rotor
- removed link RR_thigh
- removed link RR_thigh_rotor
- removed link base
- added link FL_LOWER_LEG, mass 0.154; collision cylinder length=0.12 radius=0.012; visual mesh filename=./dae/calf.dae
- added link FL_LOWER_LEG_rotor, mass 0.089
- added link FL_LOWER_LEGlower; collision cylinder length=0.065 radius=0.011
- added link FL_LOWER_LEGlower1; collision cylinder length=0.03 radius=0.0155
- added link FL_SHOULDER, mass 0.678; collision cylinder length=0.04 radius=0.046; visual mesh filename=./dae/hip.dae
- added link FL_SHOULDER_rotor, mass 0.089
- added link FL_UPPER_LEG, mass 1.152; collision box size=0.11 0.0245 0.034; visual mesh filename=./dae/thigh.dae
- added link FL_UPPER_LEG_rotor, mass 0.089
- added link FR_LOWER_LEG, mass 0.154; collision cylinder length=0.12 radius=0.013; visual mesh filename=./dae/calf_mirror.dae
- added link FR_LOWER_LEG_rotor, mass 0.089
- added link FR_LOWER_LEGlower; collision cylinder length=0.065 radius=0.011
- added link FR_LOWER_LEGlower1; collision cylinder length=0.03 radius=0.0155
- added link FR_SHOULDER, mass 0.678; collision cylinder length=0.04 radius=0.046; visual mesh filename=./dae/hip.dae
- added link FR_SHOULDER_rotor, mass 0.089
- added link FR_UPPER_LEG, mass 1.152; collision box size=0.11 0.0245 0.034; visual mesh filename=./dae/thigh_mirror.dae
- added link FR_UPPER_LEG_rotor, mass 0.089
- added link HL_LOWER_LEG, mass 0.154; collision cylinder length=0.12 radius=0.013; visual mesh filename=./dae/calf.dae
- added link HL_LOWER_LEG_rotor, mass 0.089
- added link HL_LOWER_LEGlower; collision cylinder length=0.065 radius=0.011
- added link HL_LOWER_LEGlower1; collision cylinder length=0.03 radius=0.0155
- added link HL_SHOULDER, mass 0.678; collision cylinder length=0.04 radius=0.046; visual mesh filename=./dae/hip.dae
- added link HL_SHOULDER_rotor, mass 0.089
- added link HL_UPPER_LEG, mass 1.152; collision box size=0.11 0.0245 0.034; visual mesh filename=./dae/thigh.dae
- added link HL_UPPER_LEG_rotor, mass 0.089
- added link HL_foot, mass 0.04; collision sphere radius=0.022; visual mesh filename=./dae/foot.dae
- added link HR_LOWER_LEG, mass 0.154; collision cylinder length=0.12 radius=0.013; visual mesh filename=./dae/calf_mirror.dae
- added link HR_LOWER_LEG_rotor, mass 0.089
- added link HR_LOWER_LEGlower; collision cylinder length=0.065 radius=0.011
- added link HR_LOWER_LEGlower1; collision cylinder length=0.03 radius=0.0155
- added link HR_SHOULDER, mass 0.678; collision cylinder length=0.04 radius=0.046; visual mesh filename=./dae/hip.dae
- added link HR_SHOULDER_rotor, mass 0.089
- added link HR_UPPER_LEG, mass 1.152; collision box size=0.11 0.0245 0.034; visual mesh filename=./dae/thigh_mirror.dae
- added link HR_UPPER_LEG_rotor, mass 0.089
- added link HR_foot, mass 0.04; collision sphere radius=0.022; visual mesh filename=./dae/foot.dae
- added link base_link, mass 6.921; collision box size=0.3762 0.0935 0.114; visual mesh filename=./dae/base.dae
Joints:
- removed joint FL_calf_joint
- removed joint FL_calf_rotor_joint
- removed joint FL_calflower1_joint
- removed joint FL_calflower_joint
- removed joint FL_hip_joint
- removed joint FL_hip_rotor_joint
- removed joint FL_thigh_joint
- removed joint FL_thigh_rotor_joint
- removed joint FR_calf_joint
- removed joint FR_calf_rotor_joint
- removed joint FR_calflower1_joint
- removed joint FR_calflower_joint
- removed joint FR_hip_joint
- removed joint FR_hip_rotor_joint
- removed joint FR_thigh_joint
- removed joint FR_thigh_rotor_joint
- removed joint RL_calf_joint
- removed joint RL_calf_rotor_joint
- removed joint RL_calflower1_joint
- removed joint RL_calflower_joint
- removed joint RL_foot_joint
- removed joint RL_hip_joint
- removed joint RL_hip_rotor_joint
- removed joint RL_thigh_joint
- removed joint RL_thigh_rotor_joint
- removed joint RR_calf_joint
- removed joint RR_calf_rotor_joint
- removed joint RR_calflower1_joint
- removed joint RR_calflower_joint
- removed joint RR_foot_joint
- removed joint RR_hip_joint
- removed joint RR_hip_rotor_joint
- removed joint RR_thigh_joint
- removed joint RR_thigh_rotor_joint
- added joint FL_HAA: type revolute, parent base_link, child FL_SHOULDER, origin xyz=0.1934 0.0465 0 rpy=0 0 0, axis 1 0 0, limit lower=-1.0472 upper=1.0472 effort=23.7 velocity=30.1
- added joint FL_HFE: type revolute, parent FL_SHOULDER, child FL_UPPER_LEG, origin xyz=0 0.0955 0 rpy=0 0 0, axis 0 1 0, limit lower=-1.5708 upper=3.4907 effort=23.7 velocity=30.1
- added joint FL_KFE: type revolute, parent FL_UPPER_LEG, child FL_LOWER_LEG, origin xyz=0 0 -0.213 rpy=0 0 0, axis 0 1 0, limit lower=-2.7227 upper=-0.83776 effort=45.43 velocity=15.70
- added joint FL_LOWER_LEG_rotor_joint: type fixed, parent FL_UPPER_LEG, child FL_LOWER_LEG_rotor, origin xyz=0 -0.03235 0 rpy=0 0 0
- added joint FL_LOWER_LEGlower1_joint: type fixed, parent FL_LOWER_LEGlower, child FL_LOWER_LEGlower1, origin xyz=-0.01 0 -0.04 rpy=0 0.48 0, axis 0 0 0
- added joint FL_LOWER_LEGlower_joint: type fixed, parent FL_LOWER_LEG, child FL_LOWER_LEGlower, origin xyz=0.020 0 -0.148 rpy=0 0.05 0, axis 0 0 0
- added joint FL_SHOULDER_rotor_joint: type fixed, parent base_link, child FL_SHOULDER_rotor, origin xyz=0.11215 0.04675 0 rpy=0 0 0
- added joint FL_UPPER_LEG_rotor_joint: type fixed, parent FL_SHOULDER, child FL_UPPER_LEG_rotor, origin xyz=0 -0.00015 0 rpy=0 0 0
- added joint FR_HAA: type revolute, parent base_link, child FR_SHOULDER, origin xyz=0.1934 -0.0465 0 rpy=0 0 0, axis 1 0 0, limit lower=-1.0472 upper=1.0472 effort=23.7 velocity=30.1
- added joint FR_HFE: type revolute, parent FR_SHOULDER, child FR_UPPER_LEG, origin xyz=0 -0.0955 0 rpy=0 0 0, axis 0 1 0, limit lower=-1.5708 upper=3.4907 effort=23.7 velocity=30.1
- added joint FR_KFE: type revolute, parent FR_UPPER_LEG, child FR_LOWER_LEG, origin xyz=0 0 -0.213 rpy=0 0 0, axis 0 1 0, limit lower=-2.7227 upper=-0.83776 effort=45.43 velocity=15.70
- added joint FR_LOWER_LEG_rotor_joint: type fixed, parent FR_UPPER_LEG, child FR_LOWER_LEG_rotor, origin xyz=0 0.03235 0 rpy=0 0 0
- added joint FR_LOWER_LEGlower1_joint: type fixed, parent FR_LOWER_LEGlower, child FR_LOWER_LEGlower1, origin xyz=-0.01 0 -0.04 rpy=0 0.48 0, axis 0 0 0
- added joint FR_LOWER_LEGlower_joint: type fixed, parent FR_LOWER_LEG, child FR_LOWER_LEGlower, origin xyz=0.020 0 -0.148 rpy=0 0.05 0, axis 0 0 0
- added joint FR_SHOULDER_rotor_joint: type fixed, parent base_link, child FR_SHOULDER_rotor, origin xyz=0.11215 -0.04675 0 rpy=0 0 0
- added joint FR_UPPER_LEG_rotor_joint: type fixed, parent FR_SHOULDER, child FR_UPPER_LEG_rotor, origin xyz=0 0.00015 0 rpy=0 0 0
- added joint HL_HAA: type revolute, parent base_link, child HL_SHOULDER, origin xyz=-0.1934 0.0465 0 rpy=0 0 0, axis 1 0 0, limit lower=-1.0472 upper=1.0472 effort=23.7 velocity=30.1
- added joint HL_HFE: type revolute, parent HL_SHOULDER, child HL_UPPER_LEG, origin xyz=0 0.0955 0 rpy=0 0 0, axis 0 1 0, limit lower=-0.5236 upper=4.5379 effort=23.7 velocity=30.1
- added joint HL_KFE: type revolute, parent HL_UPPER_LEG, child HL_LOWER_LEG, origin xyz=0 0 -0.213 rpy=0 0 0, axis 0 1 0, limit lower=-2.7227 upper=-0.83776 effort=45.43 velocity=15.70
- added joint HL_LOWER_LEG_rotor_joint: type fixed, parent HL_UPPER_LEG, child HL_LOWER_LEG_rotor, origin xyz=0 -0.03235 0 rpy=0 0 0
- added joint HL_LOWER_LEGlower1_joint: type fixed, parent HL_LOWER_LEGlower, child HL_LOWER_LEGlower1, origin xyz=-0.01 0 -0.04 rpy=0 0.48 0, axis 0 0 0
- added joint HL_LOWER_LEGlower_joint: type fixed, parent HL_LOWER_LEG, child HL_LOWER_LEGlower, origin xyz=0.020 0 -0.148 rpy=0 0.05 0, axis 0 0 0
- added joint HL_SHOULDER_rotor_joint: type fixed, parent base_link, child HL_SHOULDER_rotor, origin xyz=-0.11215 0.04675 0 rpy=0 0 0
- added joint HL_UPPER_LEG_rotor_joint: type fixed, parent HL_SHOULDER, child HL_UPPER_LEG_rotor, origin xyz=0 -0.00015 0 rpy=0 0 0
- added joint HL_foot_joint: type fixed, parent HL_LOWER_LEG, child HL_foot, origin xyz=0 0 -0.213 rpy=0 0 0, axis 0 0 0
- added joint HR_HAA: type revolute, parent base_link, child HR_SHOULDER, origin xyz=-0.1934 -0.0465 0 rpy=0 0 0, axis 1 0 0, limit lower=-1.0472 upper=1.0472 effort=23.7 velocity=30.1
- added joint HR_HFE: type revolute, parent HR_SHOULDER, child HR_UPPER_LEG, origin xyz=0 -0.0955 0 rpy=0 0 0, axis 0 1 0, limit lower=-0.5236 upper=4.5379 effort=23.7 velocity=30.1
- added joint HR_KFE: type revolute, parent HR_UPPER_LEG, child HR_LOWER_LEG, origin xyz=0 0 -0.213 rpy=0 0 0, axis 0 1 0, limit lower=-2.7227 upper=-0.83776 effort=45.43 velocity=15.70
- added joint HR_LOWER_LEG_rotor_joint: type fixed, parent HR_UPPER_LEG, child HR_LOWER_LEG_rotor, origin xyz=0 0.03235 0 rpy=0 0 0
- added joint HR_LOWER_LEGlower1_joint: type fixed, parent HR_LOWER_LEGlower, child HR_LOWER_LEGlower1, origin xyz=-0.01 0 -0.04 rpy=0 0.48 0, axis 0 0 0
- added joint HR_LOWER_LEGlower_joint: type fixed, parent HR_LOWER_LEG, child HR_LOWER_LEGlower, origin xyz=0.020 0 -0.148 rpy=0 0.05 0, axis 0 0 0
- added joint HR_SHOULDER_rotor_joint: type fixed, parent base_link, child HR_SHOULDER_rotor, origin xyz=-0.11215 -0.04675 0 rpy=0 0 0
- added joint HR_UPPER_LEG_rotor_joint: type fixed, parent HR_SHOULDER, child HR_UPPER_LEG_rotor, origin xyz=0 0.00015 0 rpy=0 0 0
- added joint HR_foot_joint: type fixed, parent HR_LOWER_LEG, child HR_foot, origin xyz=0 0 -0.213 rpy=0 0 0, axis 0 0 0
- joint FL_foot_joint: parent FL_calf -> FL_LOWER_LEG
- joint FR_foot_joint: parent FR_calf -> FR_LOWER_LEG
- joint Head_upper_joint: parent base -> base_link
- joint front_camera_joint: parent base -> base_link
- joint imu_joint: parent base -> base_link
- joint radar_joint: parent base -> base_link
